Commit message: change package location to absolute in iss urdf and astrobee xacro

File: src/resources/astrobee.xacro (robot description, xacro)
@@ -34,5 +34,5 @@
       <origin xyz="0 0 0" rpy="0 0 0" />
       <geometry>
-        <mesh filename="package://astrobee_freeflyer/meshes/body.dae"/>
+        <mesh filename="/home/dan/astrobee/src/description/media/astrobee_freeflyer/meshes/body.dae"/>
       </geometry>
     </visual>
@@ -47,5 +47,5 @@
       <origin xyz="0 0 0" rpy="0 0 0" />
       <geometry>
-        <mesh filename="package://astrobee_freeflyer/meshes/pmc.dae"/>
+        <mesh filename="/home/dan/astrobee/src/description/media/astrobee_freeflyer/meshes/pmc.dae"/>
       </geometry>
     </visual>
@@ -53,5 +53,5 @@
       <origin xyz="0 0 0" rpy="0 0 0" />
       <geometry>
-        <mesh filename="package://astrobee_freeflyer/meshes/pmc_bumper.dae"/>
+        <mesh filename="/home/dan/astrobee/src/description/media/astrobee_freeflyer/meshes/pmc_bumper.dae"/>
       </geometry>
     </visual>
@@ -59,5 +59,5 @@
       <origin xyz="0 0 0" rpy="0 0 0" />
       <geometry>
-        <mesh filename="package://astrobee_freeflyer/meshes/pmc_skin${ns}.dae"/>
+        <mesh filename="/home/dan/astrobee/src/description/media/astrobee_freeflyer/meshes/pmc_skin${ns}.dae"/>
       </geometry>
     </visual>
@@ -72,5 +72,5 @@
       <origin xyz="0 0 0" rpy="0 3.14 3.14" />
       <geometry>
-        <mesh filename="package://astrobee_freeflyer/meshes/pmc.dae"/>
+        <mesh filename="/home/dan/astrobee/src/description/media/astrobee_freeflyer/meshes/pmc.dae"/>
       </geometry>
     </visual>
@@ -78,5 +78,5 @@
       <origin xyz="0 0 0" rpy="0 3.14 3.14" />
       <geometry>
-        <mesh filename="package://astrobee_freeflyer/meshes/pmc_bumper.dae"/>
+        <mesh filename="/home/dan/astrobee/src/description/media/astrobee_freeflyer/meshes/pmc_bumper.dae"/>
       </geometry>
     </visual>
@@ -84,5 +84,5 @@
       <origin xyz="0 0 0" rpy="0 3.14 3.14" />
       <geometry>
-        <mesh filename="package://astrobee_freeflyer/meshes/pmc_skin${ns}.dae"/>
+        <mesh filename="/home/dan/astrobee/src/description/media/astrobee_freeflyer/meshes/pmc_skin${ns}.dae"/>
       </geometry>
     </visual>
@@ -109,22 +109,22 @@
   </joint>
   <!-- MODEL -->
-  <xacro:include filename="$(find description)/urdf/model_drag.urdf.xacro" />
-  <xacro:include filename="$(find description)/urdf/model_pmc.urdf.xacro" />
-  <xacro:include filename="$(find description)/urdf/model_eps.urdf.xacro" />
-  <xacro:include filename="$(find description)/urdf/model_truth.urdf.xacro" />
-  <xacro:include filename="$(find description)/urdf/model_laser.urdf.xacro" />
-  <xacro:include filename="$(find description)/urdf/model_flashlights.urdf.xacro" />
-  <xacro:include filename="$(find description)/urdf/model_speed_cam.urdf.xacro" />
-  <xacro:include filename="$(find description)/urdf/model_signal_lights.urdf.xacro" />
+  <xacro:include filename="/home/dan/astrobee/src/description/description/urdf/model_drag.urdf.xacro" />
+  <xacro:include filename="/home/dan/astrobee/src/description/description/urdf/model_pmc.urdf.xacro" />
+  <xacro:include filename="/home/dan/astrobee/src/description/description/urdf/model_eps.urdf.xacro" />
+  <xacro:include filename="/home/dan/astrobee/src/description/description/urdf/model_truth.urdf.xacro" />
+  <xacro:include filename="/home/dan/astrobee/src/description/description/urdf/model_laser.urdf.xacro" />
+  <xacro:include filename="/home/dan/astrobee/src/description/description/urdf/model_flashlights.urdf.xacro" />
+  <xacro:include filename="/home/dan/astrobee/src/description/description/urdf/model_speed_cam.urdf.xacro" />
+  <xacro:include filename="/home/dan/astrobee/src/description/description/urdf/model_signal_lights.urdf.xacro" />
   <!-- Monitors -->
-  <xacro:include filename="$(find description)/urdf/model_monitors.urdf.xacro" />
+  <xacro:include filename="/home/dan/astrobee/src/description/description/urdf/model_monitors.urdf.xacro" />
   <!-- SENSORS -->
-  <xacro:include filename="$(find description)/urdf/sensor_imu.urdf.xacro" />
-  <xacro:include filename="$(find description)/urdf/sensor_nav_cam.urdf.xacro" />
-  <xacro:include filename="$(find description)/urdf/sensor_dock_cam.urdf.xacro" />
-  <xacro:include filename="$(find description)/urdf/sensor_haz_cam.urdf.xacro" />
-  <xacro:include filename="$(find description)/urdf/sensor_perch_cam.urdf.xacro" />
+  <xacro:include filename="/home/dan/astrobee/src/description/description/urdf/sensor_imu.urdf.xacro" />
+  <xacro:include filename="/home/dan/astrobee/src/description/description/urdf/sensor_nav_cam.urdf.xacro" />
+  <xacro:include filename="/home/dan/astrobee/src/description/description/urdf/sensor_dock_cam.urdf.xacro" />
+  <xacro:include filename="/home/dan/astrobee/src/description/description/urdf/sensor_haz_cam.urdf.xacro" />
+  <xacro:include filename="/home/dan/astrobee/src/description/description/urdf/sensor_perch_cam.urdf.xacro" />
   <!-- PERCHING ARM -->
-  <xacro:include filename="$(find description)/urdf/macro_perching_arm.urdf.xacro" />
+  <xacro:include filename="/home/dan/astrobee/src/description/description/urdf/macro_perching_arm.urdf.xacro" />
   <xacro:if value="${pay_top_aft == 'perching_arm'}">
     <xacro:perching_arm bay="top_aft"
@@ -144,5 +144,5 @@
   <!-- GRANITE-SPECIFIC OPTIONS -->
   <xacro:if value="${world == 'granite'}">
-    <xacro:include filename="$(find description)/urdf/model_carriage.urdf.xacro" />
+    <xacro:include filename="/home/dan/astrobee/src/description/description/urdf/model_carriage.urdf.xacro" />
   </xacro:if>
 </robot>

File: src/resources/iss.urdf (robot description, URDF)
Before this commit: robot iss, 1 links, 0 joints
Links:
- link body: geometry collision mesh filename=/home/dan/astrobee/src/description/media/astrobee_iss/meshe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; collision mesh filename=/home/dan/astrobee/src/description/media/astrobee_iss/meshe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
