Commit message: had to manually modify the astrobee urdf to get it to work

File: src/resources/astrobee.urdf (robot description, URDF)
Before this commit: robot astrobee, 9 links, 8 joints
Links:
- removed link honeybody
- removed link honeyinertial_link
- removed link honeytop_aft
- removed link honeytop_aft_arm_distal_link
- removed link honeytop_aft_arm_proximal_link
- removed link honeytop_aft_gripper_left_distal_link
- removed link honeytop_aft_gripper_left_proximal_link
- removed link honeytop_aft_gripper_right_distal_link
- removed link honeytop_aft_gripper_right_proximal_link
- added link honey_body; collision box size=0.290513 0.151942 0.281129; collision box size=0.319199 0.083962 0.319588
- added link honey_inertial_link, mass 9.0877
- added link honey_top_aft, mass 0.3078; collision box size=0.090441 0.152400 0.076250; visual mesh filename=/home/dan/astrobee/src/description/media/astrobee_freeflyer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
- added link honey_top_aft_arm_distal_link, mass 0.1033; collision box size=0.075000 0.070000 0.087400; visual mesh filename=/home/dan/astrobee/src/description/media/astrobee_freeflyer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
- added link honey_top_aft_arm_proximal_link, mass 0.1623; collision box size=0.123250 0.068000 0.042400; visual mesh filename=/home/dan/astrobee/src/description/media/astrobee_freeflyer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
- added link honey_top_aft_gripper_left_distal_link, mass 0.0116026396896178; collision box size=0.056953 0.021750 0.025400; visual mesh filename=/home/dan/astrobee/src/description/media/astrobee_freeflyer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
- added link honey_top_aft_gripper_left_proximal_link, mass 0.04; collision box size=0.067654 0.021750 0.025400; visual mesh filename=/home/dan/astrobee/src/description/media/astrobee_freeflyer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
- added link honey_top_aft_gripper_right_distal_link, mass 0.02285; collision box size=0.056894 0.021750 0.025400; visual mesh filename=/home/dan/astrobee/src/description/media/astrobee_freeflyer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
- added link honey_top_aft_gripper_right_proximal_link, mass 0.04; collision box size=0.067654 0.021750 0.025400; visual mesh filename=/home/dan/astrobee/src/description/media/astrobee_freeflyer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
Joints:
- joint inertial_joint: child honeyinertial_link -> honey_inertial_link; parent honeybody -> honey_body
- joint top_aft: child honeytop_aft -> honey_top_aft; parent honeybody -> honey_body
- joint top_aft_arm_distal_joint: child honeytop_aft_arm_distal_link -> honey_top_aft_arm_distal_link; parent honeytop_aft_arm_proximal_link -> honey_top_aft_arm_proximal_link
- joint top_aft_arm_proximal_joint: child honeytop_aft_arm_proximal_link -> honey_top_aft_arm_proximal_link; parent honeytop_aft -> honey_top_aft
- joint top_aft_gripper_left_distal_joint: child honeytop_aft_gripper_left_distal_link -> honey_top_aft_gripper_left_distal_link; parent honeytop_aft_gripper_left_proximal_link -> honey_top_aft_gripper_left_proximal_link
- joint top_aft_gripper_left_proximal_joint: child honeytop_aft_gripper_left_proximal_link -> honey_top_aft_gripper_left_proximal_link; parent honeytop_aft_arm_distal_link -> honey_top_aft_arm_distal_link
- joint top_aft_gripper_right_distal_joint: child honeytop_aft_gripper_right_distal_link -> honey_top_aft_gripper_right_distal_link; parent honeytop_aft_gripper_right_proximal_link -> honey_top_aft_gripper_right_proximal_link
- joint top_aft_gripper_right_proximal_joint: child honeytop_aft_gripper_right_proximal_link -> honey_top_aft_gripper_right_proximal_link; parent honeytop_aft_arm_distal_link -> honey_top_aft_arm_distal_link
