Commit message: update the ISS urdf to use VHACD for collision info, add debugging version

File: src/resources/iss_collision.urdf (robot description, URDF)
Before this commit: robot iss, 1 links, 0 joints
Links:
- link body: geometry collision mesh filename=/home/dan/astrobee_pybullet/src/resources/iss_objs/vhacd_re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; collision mesh filename=/home/dan/astrobee_pybullet/src/resources/iss_objs/vhacd_re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

File: src/resources/iss_original.urdf (robot description, URDF)
Before this commit: robot iss, 1 links, 0 joints
Links:
- link body: geometry collision mesh filename=/home/dan/astrobee/src/description/media/astrobee_iss/meshe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; collision mesh filename=/home/dan/astrobee/src/description/media/astrobee_iss/meshe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
