Commit message: change filenames in iss urdf to outside of catkin package

File: src/resources/iss.urdf (robot description, URDF)
Before this commit: robot iss, 1 links, 0 joints
Links:
- link body: geometry collision mesh filename=$HOME/astrobee/src/description/media/astrobee_iss/meshes/cu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; collision mesh filename=$HOME/astrobee/src/description/media/astrobee_iss/meshes/eu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

Commit message: Update cargo bag mesh and reorganize mesh files

File: src/resources/iss.urdf (robot description, URDF)
Before this commit: robot iss, 1 links, 0 joints
Links:
- link body: geometry collision mesh filename=/home/dan/astrobee_pybullet/src/resources/meshes/vhacd/eu_l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; collision mesh filename=/home/dan/astrobee_pybullet/src/resources/meshes/vhacd/jpm.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

File: src/resources/iss_collision.urdf (robot description, URDF)
Before this commit: robot iss, 1 links, 0 joints
Links:
- link body: geometry collision mesh filename=/home/dan/astrobee_pybullet/src/resources/meshes/vhacd/eu_l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; collision mesh filename=/home/dan/astrobee_pybullet/src/resources/meshes/vhacd/jpm.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
