Commit message: change remaining instances of src to astrobee_pybullet

File: astrobee_pybullet/resources/urdf/cargo_bag_rigid.urdf (robot description, URDF)
Before this commit: robot bag, 1 links, 0 joints
Links:
- link baseLink: geometry collision mesh filename=/home/dan/astrobee_pybullet/astrobee_pybullet/resources/mes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 scale=1 1 1; visual mesh filename=/home/dan/astrobee_pybullet/astrobee_pybullet/resources/mes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 scale=1 1 1

File: astrobee_pybullet/resources/urdf/iss.urdf (robot description, URDF)
Before this commit: robot iss, 1 links, 0 joints
Links:
- link body: geometry collision mesh filename=/home/dan/astrobee_pybullet/astrobee_pybullet/resources/mes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; collision mesh filename=/home/dan/astrobee_pybullet/astrobee_pybullet/resources/mes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

File: astrobee_pybullet/resources/urdf/iss_collision.urdf (robot description, URDF)
Before this commit: robot iss, 1 links, 0 joints
Links:
- link body: geometry collision mesh filename=/home/dan/astrobee_pybullet/astrobee_pybullet/resources/mes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; collision mesh filename=/home/dan/astrobee_pybullet/astrobee_pybullet/resources/mes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
