Commit message: remove their KDL inertia workaround so pybullet can read it properly

File: astrobee_pybullet/resources/urdf/astrobee_2.urdf (robot description, URDF)
Before this commit: robot astrobee, 9 links, 8 joints
Links:
- removed link honey_inertial_link
- link honey_body: mass None -> 9.0877
Joints:
- removed joint inertial_joint
