Commit message: Update meshes and textures to get Astrobee to load with proper visuals

File: pyastrobee/assets/urdf/astrobee.urdf (robot description, URDF)
Before this commit: robot astrobee, 8 links, 7 joints
Links:
- link honey_body: geometry collision box size=0.290513 0.151942 0.281129; collision box size=0.319199 0.083962 0.319588
- link honey_top_aft: geometry collision box size=0.090441 0.152400 0.076250; visual mesh filename=../meshes/astrobee/base_link.obj
- link honey_top_aft_arm_distal_link: geometry collision box size=0.075000 0.070000 0.087400; visual mesh filename=../meshes/astrobee/arm_distal_link.obj
- link honey_top_aft_arm_proximal_link: geometry collision box size=0.123250 0.068000 0.042400; visual mesh filename=../meshes/astrobee/arm_proximal_link.obj
- link honey_top_aft_gripper_left_distal_link: geometry collision box size=0.056953 0.021750 0.025400; visual mesh filename=../meshes/astrobee/gripper_left_distal_link.obj
- link honey_top_aft_gripper_left_proximal_link: geometry collision box size=0.067654 0.021750 0.025400; visual mesh filename=../meshes/astrobee/gripper_left_proximal_link.obj
- link honey_top_aft_gripper_right_distal_link: geometry collision box size=0.056894 0.021750 0.025400; visual mesh filename=../meshes/astrobee/gripper_right_distal_link.obj
- link honey_top_aft_gripper_right_proximal_link: geometry collision box size=0.067654 0.021750 0.025400; visual mesh filename=../meshes/astrobee/gripper_right_proximal_link.obj
