Commit message: Update folder for bag OBJ meshes

File: pyastrobee/assets/urdf/astrobee_with_rigid_bag.urdf (robot description, URDF)
Before this commit: robot astrobee, 9 links, 8 joints
Links:
- link bag: geometry collision box size=0.50 0.25 0.42; visual mesh filename=../meshes/bags/top_handle_bag.obj

Commit message: Update bag names for consistency

File: pyastrobee/assets/urdf/astrobee_with_rigid_bag.urdf (robot description, URDF)
Before this commit: robot astrobee, 9 links, 8 joints
Links:
- link bag: geometry collision box size=0.50 0.25 0.42; visual mesh filename=../meshes/bags/top_handle.obj
