Commit message: update handle position to match transforms from original bag

File: pyastrobee/assets/urdf/rigid_bag.urdf (robot description, URDF)
Before this commit: robot cargo_bag, 5 links, 4 joints
Joints:
- joint handle_joint: origin xyz=0 0 0.025 -> xyz=0 0 0.035

Commit message: Split the collision info into 3 to add empty region around handle

File: pyastrobee/assets/urdf/rigid_bag.urdf (robot description, URDF)
Before this commit: robot cargo_bag, 5 links, 4 joints
Links:
- link main_compartment_link: geometry collision box size=0.15 0.25 0.42; collision box size=0.15 0.25 0.42
