Commit message: Support for all single-handle rigid bags

File: pyastrobee/assets/urdf/right_handle_rigid_bag.urdf (robot description, URDF)
Before this commit: robot cargo_bag, 5 links, 4 joints
Links:
- link handle_link: geometry collision box size=0.02 0.05 0.15; visual box size=0.02 0.05 0.15
- link main_compartment_link: geometry collision box size=0.44 0.25 0.20; collision box size=0.50 0.25 0.11
Joints:
- joint handle_joint: origin xyz=0 0 0.035 -> xyz=0.035 0 0 rpy=0 0 0
- joint pitch_joint: origin xyz=0 0 0.21 rpy=0 0 0 -> xyz=0.25 0 0 rpy=0 0 0
