Commit message: Update bag handle: Reduce collision size, increase angular limits

File: pyastrobee/assets/urdf/bags/front_back_handle_rigid_bag.urdf (robot description, URDF)
Before this commit: robot cargo_bag, 9 links, 8 joints
Links:
- link handle_link: geometry collision box size=0.02 0.05 0.05; visual box size=0.02 0.05 0.15
Joints:
- joint pitch_joint: limit lower=-0.7 upper=0.7 effort=1.0 velocity=1.0 -> lower=-1.57079 upper=1.57079 effort=1.0 velocity=1.0
- joint pitch_joint_2: limit lower=-0.7 upper=0.7 effort=1.0 velocity=1.0 -> lower=-1.57079 upper=1.57079 effort=1.0 velocity=1.0
- joint roll_joint: limit lower=-0.52360 upper=0.52360 effort=1.0 velocity=1.0 -> lower=-1.57079 upper=1.57079 effort=1.0 velocity=1.0
- joint roll_joint_2: limit lower=-0.52360 upper=0.52360 effort=1.0 velocity=1.0 -> lower=-1.57079 upper=1.57079 effort=1.0 velocity=1.0
- joint yaw_joint: limit lower=-0.52360 upper=0.52360 effort=1.0 velocity=1.0 -> lower=-1.57079 upper=1.57079 effort=1.0 velocity=1.0
- joint yaw_joint_2: limit lower=-0.52360 upper=0.52360 effort=1.0 velocity=1.0 -> lower=-1.57079 upper=1.57079 effort=1.0 velocity=1.0

File: pyastrobee/assets/urdf/bags/front_handle_rigid_bag.urdf (robot description, URDF)
Before this commit: robot cargo_bag, 5 links, 4 joints
Links:
- link handle_link: geometry collision box size=0.02 0.05 0.05; visual box size=0.02 0.05 0.15
Joints:
- joint pitch_joint: limit lower=-0.7 upper=0.7 effort=1.0 velocity=1.0 -> lower=-1.57079 upper=1.57079 effort=1.0 velocity=1.0
- joint roll_joint: limit lower=-0.52360 upper=0.52360 effort=1.0 velocity=1.0 -> lower=-1.57079 upper=1.57079 effort=1.0 velocity=1.0
- joint yaw_joint: limit lower=-0.52360 upper=0.52360 effort=1.0 velocity=1.0 -> lower=-1.57079 upper=1.57079 effort=1.0 velocity=1.0

File: pyastrobee/assets/urdf/bags/right_handle_rigid_bag.urdf (robot description, URDF)
Before this commit: robot cargo_bag, 5 links, 4 joints
Links:
- link handle_link: geometry collision box size=0.02 0.05 0.05; visual box size=0.02 0.05 0.15
Joints:
- joint pitch_joint: limit lower=-0.7 upper=0.7 effort=1.0 velocity=1.0 -> lower=-1.57079 upper=1.57079 effort=1.0 velocity=1.0
- joint roll_joint: limit lower=-0.52360 upper=0.52360 effort=1.0 velocity=1.0 -> lower=-1.57079 upper=1.57079 effort=1.0 velocity=1.0
- joint yaw_joint: limit lower=-0.52360 upper=0.52360 effort=1.0 velocity=1.0 -> lower=-1.57079 upper=1.57079 effort=1.0 velocity=1.0

File: pyastrobee/assets/urdf/bags/right_left_handle_rigid_bag.urdf (robot description, URDF)
Before this commit: robot cargo_bag, 9 links, 8 joints
Links:
- link handle_link: geometry collision box size=0.02 0.05 0.05; visual box size=0.02 0.05 0.15
Joints:
- joint pitch_joint: limit lower=-0.7 upper=0.7 effort=1.0 velocity=1.0 -> lower=-1.57079 upper=1.57079 effort=1.0 velocity=1.0
- joint pitch_joint_2: limit lower=-0.7 upper=0.7 effort=1.0 velocity=1.0 -> lower=-1.57079 upper=1.57079 effort=1.0 velocity=1.0
- joint roll_joint: limit lower=-0.52360 upper=0.52360 effort=1.0 velocity=1.0 -> lower=-1.57079 upper=1.57079 effort=1.0 velocity=1.0
- joint roll_joint_2: limit lower=-0.52360 upper=0.52360 effort=1.0 velocity=1.0 -> lower=-1.57079 upper=1.57079 effort=1.0 velocity=1.0
- joint yaw_joint: limit lower=-0.52360 upper=0.52360 effort=1.0 velocity=1.0 -> lower=-1.57079 upper=1.57079 effort=1.0 velocity=1.0
- joint yaw_joint_2: limit lower=-0.52360 upper=0.52360 effort=1.0 velocity=1.0 -> lower=-1.57079 upper=1.57079 effort=1.0 velocity=1.0

File: pyastrobee/assets/urdf/bags/top_bottom_handle_rigid_bag.urdf (robot description, URDF)
Before this commit: robot cargo_bag, 9 links, 8 joints
Links:
- link handle_link: geometry collision box size=0.02 0.05 0.05; visual box size=0.02 0.05 0.15
Joints:
- joint pitch_joint: limit lower=-0.7 upper=0.7 effort=1.0 velocity=1.0 -> lower=-1.57079 upper=1.57079 effort=1.0 velocity=1.0
- joint pitch_joint_2: limit lower=-0.7 upper=0.7 effort=1.0 velocity=1.0 -> lower=-1.57079 upper=1.57079 effort=1.0 velocity=1.0
- joint roll_joint: limit lower=-0.52360 upper=0.52360 effort=1.0 velocity=1.0 -> lower=-1.57079 upper=1.57079 effort=1.0 velocity=1.0
- joint roll_joint_2: limit lower=-0.52360 upper=0.52360 effort=1.0 velocity=1.0 -> lower=-1.57079 upper=1.57079 effort=1.0 velocity=1.0
- joint yaw_joint: limit lower=-0.52360 upper=0.52360 effort=1.0 velocity=1.0 -> lower=-1.57079 upper=1.57079 effort=1.0 velocity=1.0
- joint yaw_joint_2: limit lower=-0.52360 upper=0.52360 effort=1.0 velocity=1.0 -> lower=-1.57079 upper=1.57079 effort=1.0 velocity=1.0

File: pyastrobee/assets/urdf/bags/top_handle_rigid_bag.urdf (robot description, URDF)
Before this commit: robot cargo_bag, 5 links, 4 joints
Links:
- link handle_link: geometry collision box size=0.02 0.05 0.05; visual box size=0.02 0.05 0.15
Joints:
- joint pitch_joint: limit lower=-0.7 upper=0.7 effort=1.0 velocity=1.0 -> lower=-1.57079 upper=1.57079 effort=1.0 velocity=1.0
- joint roll_joint: limit lower=-0.52360 upper=0.52360 effort=1.0 velocity=1.0 -> lower=-1.57079 upper=1.57079 effort=1.0 velocity=1.0
- joint yaw_joint: limit lower=-0.52360 upper=0.52360 effort=1.0 velocity=1.0 -> lower=-1.57079 upper=1.57079 effort=1.0 velocity=1.0

Commit message: Update bag handle: Reduce collision size, increase angular limits (#15)

File: pyastrobee/assets/urdf/bags/front_back_handle_rigid_bag.urdf (robot description, URDF)
Before this commit: robot cargo_bag, 9 links, 8 joints
Links:
- link handle_link: geometry collision box size=0.02 0.05 0.05; visual box size=0.02 0.05 0.15
- link handle_link_2: geometry collision box size=0.02 0.05 0.05; visual box size=0.02 0.05 0.15
Joints:
- joint pitch_joint: limit lower=-0.7 upper=0.7 effort=1.0 velocity=1.0 -> lower=-1.57079 upper=1.57079 effort=1.0 velocity=1.0
- joint pitch_joint_2: limit lower=-0.7 upper=0.7 effort=1.0 velocity=1.0 -> lower=-1.57079 upper=1.57079 effort=1.0 velocity=1.0
- joint roll_joint: limit lower=-0.52360 upper=0.52360 effort=1.0 velocity=1.0 -> lower=-1.57079 upper=1.57079 effort=1.0 velocity=1.0
- joint roll_joint_2: limit lower=-0.52360 upper=0.52360 effort=1.0 velocity=1.0 -> lower=-1.57079 upper=1.57079 effort=1.0 velocity=1.0
- joint yaw_joint: limit lower=-0.52360 upper=0.52360 effort=1.0 velocity=1.0 -> lower=-1.57079 upper=1.57079 effort=1.0 velocity=1.0
- joint yaw_joint_2: limit lower=-0.52360 upper=0.52360 effort=1.0 velocity=1.0 -> lower=-1.57079 upper=1.57079 effort=1.0 velocity=1.0

File: pyastrobee/assets/urdf/bags/right_left_handle_rigid_bag.urdf (robot description, URDF)
Before this commit: robot cargo_bag, 9 links, 8 joints
Links:
- link handle_link: geometry collision box size=0.02 0.05 0.05; visual box size=0.02 0.05 0.15
- link handle_link_2: geometry collision box size=0.02 0.05 0.05; visual box size=0.02 0.05 0.15
Joints:
- joint pitch_joint: limit lower=-0.7 upper=0.7 effort=1.0 velocity=1.0 -> lower=-1.57079 upper=1.57079 effort=1.0 velocity=1.0
- joint pitch_joint_2: limit lower=-0.7 upper=0.7 effort=1.0 velocity=1.0 -> lower=-1.57079 upper=1.57079 effort=1.0 velocity=1.0
- joint roll_joint: limit lower=-0.52360 upper=0.52360 effort=1.0 velocity=1.0 -> lower=-1.57079 upper=1.57079 effort=1.0 velocity=1.0
- joint roll_joint_2: limit lower=-0.52360 upper=0.52360 effort=1.0 velocity=1.0 -> lower=-1.57079 upper=1.57079 effort=1.0 velocity=1.0
- joint yaw_joint: limit lower=-0.52360 upper=0.52360 effort=1.0 velocity=1.0 -> lower=-1.57079 upper=1.57079 effort=1.0 velocity=1.0
- joint yaw_joint_2: limit lower=-0.52360 upper=0.52360 effort=1.0 velocity=1.0 -> lower=-1.57079 upper=1.57079 effort=1.0 velocity=1.0

File: pyastrobee/assets/urdf/bags/top_bottom_handle_rigid_bag.urdf (robot description, URDF)
Before this commit: robot cargo_bag, 9 links, 8 joints
Links:
- link handle_link: geometry collision box size=0.02 0.05 0.05; visual box size=0.02 0.05 0.15
- link handle_link_2: geometry collision box size=0.02 0.05 0.05; visual box size=0.02 0.05 0.15
Joints:
- joint pitch_joint: limit lower=-0.7 upper=0.7 effort=1.0 velocity=1.0 -> lower=-1.57079 upper=1.57079 effort=1.0 velocity=1.0
- joint pitch_joint_2: limit lower=-0.7 upper=0.7 effort=1.0 velocity=1.0 -> lower=-1.57079 upper=1.57079 effort=1.0 velocity=1.0
- joint roll_joint: limit lower=-0.52360 upper=0.52360 effort=1.0 velocity=1.0 -> lower=-1.57079 upper=1.57079 effort=1.0 velocity=1.0
- joint roll_joint_2: limit lower=-0.52360 upper=0.52360 effort=1.0 velocity=1.0 -> lower=-1.57079 upper=1.57079 effort=1.0 velocity=1.0
- joint yaw_joint: limit lower=-0.52360 upper=0.52360 effort=1.0 velocity=1.0 -> lower=-1.57079 upper=1.57079 effort=1.0 velocity=1.0
- joint yaw_joint_2: limit lower=-0.52360 upper=0.52360 effort=1.0 velocity=1.0 -> lower=-1.57079 upper=1.57079 effort=1.0 velocity=1.0
